File: hw/Lab3_Schematic.kicad_sch (KiCad schematic)
At the start: 11 parts, among them Q101 IRLD024PBF, SW101 UP, SW102 DOWN, SW103 LEFT, SW104 RIGHT, SW105 MODE, U101 EK-TM4C123GXL, U103 Adafruit ST7735R

Commit message: Changes to report and schematic
Parts:
- removed SW101: UP, Button_Switch_THT:SW_PUSH_6mm, symbol Switch:SW_Push
Connections:
- net PC5: no longer SW104.2
- net PC6: no longer SW103.2
- net PC7: no longer SW102.2
- net PF0: now also SW102.2
- net PF1: now also SW103.2
- net PF2: now also SW104.2
- net PF3: now also SW105.2
- net PF4: no longer SW105.2

Commit message: Code after Prep
Parts:
- SW102: value DOWN -> SetTime
- SW103: value LEFT -> SetAlarm
- SW104: value RIGHT -> AlarmOff
- SW105: value MODE -> DisplayMode
Connections:
- net PF0: no longer SW102.2
- net PF1: now also SW102.2; no longer SW103.2
- net PF2: now also SW103.2; no longer SW104.2
- net PF3: now also SW104.2; no longer SW105.2
- net PF4: now also SW105.2
Other:
- moved on the sheet: SW102, SW103, SW104
